Commit message: Remove unneeded components from iiwa urdf

File: frax/assets/iiwa/iiwa14.urdf (robot description, URDF)
Before this commit: robot None, 10 links, 10 joints
Links:
- removed link iiwa_link_ee
- removed link iiwa_link_ee_kuka
Joints:
- removed joint iiwa_joint_ee
- removed joint iiwa_tool0_joint
- removed joint iiwa_world_joint

Commit message: Iiwa loads (in pybullet) with visual and collision meshes based on bullet/drake

File: frax/assets/iiwa/iiwa14.urdf (robot description, URDF)
Before this commit: robot iiwa14, 8 links, 7 joints
Links:
- link iiwa_link_0: geometry collision mesh filename=../../../assets/iiwa/collision/link_0.obj; visual mesh filename=../../../assets/iiwa/visual/link_0.obj
- link iiwa_link_1: geometry collision mesh filename=../../../assets/iiwa/collision/link_1.obj; visual mesh filename=../../../assets/iiwa/visual/link_1.obj
- link iiwa_link_2: geometry collision mesh filename=../../../assets/iiwa/collision/link_2.obj; visual mesh filename=../../../assets/iiwa/visual/link_2.obj
- link iiwa_link_3: geometry collision mesh filename=../../../assets/iiwa/collision/link_3.obj; visual mesh filename=../../../assets/iiwa/visual/link_3.obj
- link iiwa_link_4: geometry collision mesh filename=../../../assets/iiwa/collision/link_4.obj; visual mesh filename=../../../assets/iiwa/visual/link_4.obj
- link iiwa_link_5: geometry collision mesh filename=../../../assets/iiwa/collision/link_5.obj; visual mesh filename=../../../assets/iiwa/visual/link_5.obj
- link iiwa_link_6: geometry collision mesh filename=../../../assets/iiwa/collision/link_6.obj; visual mesh filename=../../../assets/iiwa/visual/link_6.obj
- link iiwa_link_7: geometry collision mesh filename=../../../assets/iiwa/collision/link_7.obj; visual mesh filename=../../../assets/iiwa/visual/link_7.obj
